File: Carrier Board.sch (EAGLE design)
At the start: 54 parts, among them J1 H4P-SMD-2.0, J2 H4P-SMD-2.0, J4 S2B-PH-SM4-TB(LF)(SN), J5 S2B-PH-SM4-TB(LF)(SN), Q1 MMBT2222A, SW2 MF-SW-TACT-6MM, U1 TMP36GRTZ, U2 TPL5010, U3 MB85RC64, U7 NAND

Commit message: Had to move the Done pin to A3
Connections:
- removed net A3: BORON/ARGON/XENON.A3
- net DONE: now also BORON/ARGON/XENON.A3; no longer BORON/ARGON/XENON.D5
Changed lines of the file:
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@@
 <?xml version="1.0" encoding="utf-8"?>
 <!DOCTYPE eagle SYSTEM "eagle.dtd">
-<eagle version="9.3.2">
+<eagle version="9.4.0">
 <drawing>
 <settings>
@@
 </segment>
 </net>
-<net name="A3" class="0">
-<segment>
-<pinref part="BORON/ARGON/XENON" gate="G$1" pin="A3"/>
-<wire x1="157.48" y1="132.08" x2="149.86" y2="132.08" width="0.1524" layer="91"/>
-<label x="152.4" y="132.08" size="1.778" layer="95"/>
-</segment>
-</net>
 <net name="A2" class="0">
 <segment>
@@
 </segment>
 <segment>
-<pinref part="BORON/ARGON/XENON" gate="G$1" pin="D5"/>
-<wire x1="193.04" y1="116.84" x2="200.66" y2="116.84" width="0.1524" layer="91"/>
-<label x="200.66" y="116.84" size="1.778" layer="95" align="bottom-right"/>
-</segment>
-</net>
+<pinref part="BORON/ARGON/XENON" gate="G$1" pin="A3"/>
+<wire x1="157.48" y1="132.08" x2="149.86" y2="132.08" width="0.1524" layer="91"/>
+<label x="149.86" y="132.08" size="1.778" layer="95"/>
+</segment>
+</net>
